File: Breeze.kicad_pcb (KiCad board)
At the start: 2 copper layers, 210.6 x 114.9 mm, 102 parts, among them J1 PJ-320A, SW1 CHOCXHSPCB-1U, SW10 CHOCXHSPCB-1U, SW11 CHOCXHSPCB-1U, SW12 CHOCXHSPCB-1U, SW13 CHOCXHSPCB-1U, SW14 CHOCXHSPCB-1U, SW15 CHOCXHSPCB-1U, SW16 CHOCXHSPCB-1U, SW17 CHOCXHSPCB-1U, SW18 CHOCXHSPCB-1U, SW19 CHOCXHSPCB-1U, SW2 CHOCXHSPCB-1U, SW20 CHOCXHSPCB-1U, SW21 CHOCXHSPCB-1U, SW22 CHOCXHSPCB-1U, SW23 CHOCXHSPCB-1U, SW24 CHOCXHSPCB-1U, SW3 CHOCXHSPCB-1U, SW4 CHOCXHSPCB-1U, SW5 CHOCXHSPCB-1U, SW6 CHOCXHSPCB-1U, SW7 CHOCXHSPCB-1U, SW8 CHOCXHSPCB-1U, SW9 CHOCXHSPCB-1U

Commit message: added encoder and oled display via elite-pi
Parts:
- added J2: Conn_01x05_Pin, Connector_PinHeader_2.54mm:PinHeader_1x05_P2.54mm_Vertical, F.Cu at (120.9, 152.9)
- added J3: Conn_01x04_Socket, Connector_PinHeader_2.54mm:PinHeader_1x04_P2.54mm_Vertical, F.Cu at (122.0, 156.7)
- added SW25: RotaryEncoder_Switch, Rotary_Encoder:RotaryEncoder_Alps_EC11E-Switch_Vertical_H20mm, F.Cu at (117.5, 163.4)
- added U1: STM32H723ZGI6, STM32BGA:UFBGA-144_7X7_STM, F.Cu at (3.86, 3.86)
- moved LGO1 20.2 mm to (120.9, 176.3)
- moved RSW1 4.94 mm to (114.6, 158.0), turned to -150 degrees
- renumbered DOWN to DOWN1, LEFT to LEFT1, RIGHT to RIGHT1, UP to UP1
Connections:
- MCU-MACRO1 pad 10: Net-(MCU-MACRO1-Pad10) -> unconnected-(MCU-MACRO1-VCC-Pad10)
- MCU-MACRO1 pad 7: Net-(MCU-MACRO1-Pad7) -> unconnected-(MCU-MACRO1-RAW-Pad7)
- MCU-MAIN1 pad 1: Net-(MCU-MAIN1-Pad1) -> unconnected-(MCU-MAIN1-TX(PD3)-Pad1)
- MCU-MAIN1 pad 13: Net-(MCU-MAIN1-Pad13) -> Enc_SW
- MCU-MAIN1 pad 24: Net-(MCU-MAIN1-Pad24) -> unconnected-(MCU-MAIN1-RAW-Pad24)
- MCU-MAIN1 pad 3: GND -> Enc_A
- MCU-MAIN1 pad 4: GND -> Enc_B
Routing:
- net Enc_A: track 0.00 -> 85.1 mm, vias 0 -> 1
- net Enc_B: track 0.00 -> 74.4 mm, vias 0 -> 1
- net Enc_SW: track 0.00 -> 35.9 mm
- net GND: track 408.5 -> 386.3 mm, vias 8 -> 5
- net unconnected-(MCU-MAIN1-TX(PD3)-Pad1): track 0.00 -> 17.0 mm, vias 0 -> 1
- net Net-(MCU-MAIN1-Pad1): track 17.0 -> 0.00 mm, vias 1 -> 0
- net Net-(MCU-MAIN1-Pad13): track 14.7 -> 0.00 mm
- net unconnected-(MCU-MAIN1-RAW-Pad24): track 0.00 -> 14.4 mm
- net Net-(MCU-MAIN1-Pad24): track 14.4 -> 0.00 mm
- net Net-(J2-Pin_1): track 0.00 -> 11.3 mm
- net VCC: track 74.8 -> 83.6 mm, vias 3 -> 2
- net Net-(J2-Pin_2): track 0.00 -> 5.30 mm
- net RST: track 50.2 -> 50.7 mm
